File: back.brd (EAGLE design)
At the start: 100 x 80 mm, 26 parts, among them IC2 74AHC1G125DBV, IC3 74AHC1G125DBV, M1 HX1, X1 BU-SMA-V

Commit message: New Volt Reg Lib
Parts:
- moved JP3 497.8 mm to (-69.8, -349.2)
- moved JP2 489.1 mm to (-69.8, -340.4)
- moved JP1 480.4 mm to (-69.8, -331.5)
- moved MPU 471.5 mm to (-68.6, -326.4)
- moved IC3 464.4 mm to (-71.1, -316.2)
- moved C7 462.5 mm to (-47.0, -308.6)
- moved IC2 454.8 mm to (-62.2, -306.1)
- moved L4 438.1 mm to (-41.9, -289.6)
- moved X1 434.1 mm to (-53.3, -303.5)
- moved L3 432.4 mm to (-41.9, -284.5)
- moved C5 423.1 mm to (-39.4, -269.2)
- moved C6 423.1 mm to (-43.2, -269.2)
- moved C1 423.0 mm to (-24.1, -269.2)
- moved C2 423.0 mm to (-27.9, -269.2)
- moved C3 423.0 mm to (-31.8, -269.2)
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