File: Main.sch (EAGLE design)
At the start: 1 part

Commit message: Schematics
Parts:
- added U$1: MS5611QFN, SHC:MS5611QFN
- added U$2: M10382-A1, SHC:M10382-A1
- added U$3, U$4, U$5, U$6, U$7, U$8: 123_BATTERY_HOLDERCR-123-A, SHC:123_BATTERY_HOLDERCR-123-A
Changed lines of the file:
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@@
 <setting verticaltext="up"/>
 </settings>
-<grid distance="0.1" unitdist="inch" unit="inch" style="lines" multiple="1" display="no" altdistance="0.01" altunitdist="inch" altunit="inch"/>
+<grid distance="0.1" unitdist="inch" unit="inch" style="lines" multiple="1" display="yes" altdistance="0.01" altunitdist="inch" altunit="inch"/>
 <layers>
 <layer number="1" name="Top" color="4" fill="1" visible="no" active="no"/>
@@
 <layer number="48" name="Document" color="7" fill="1" visible="no" active="no"/>
 <layer number="49" name="Reference" color="7" fill="1" visible="no" active="no"/>
+<layer number="50" name="dxf" color="7" fill="1" visible="no" active="no"/>
 <layer number="51" name="tDocu" color="6" fill="1" visible="no" active="no"/>
 <layer number="52" name="bDocu" color="6" fill="1" visible="no" active="no"/>
+<layer number="53" name="tGND_GNDA" color="7" fill="9" visible="no" active="no"/>
+<layer number="54" name="bGND_GNDA" color="1" fill="9" visible="no" active="no"/>
+<layer number="56" name="wert" color="7" fill="1" visible="no" active="no"/>
 <layer number="90" name="Modules" color="5" fill="1" visible="yes" active="yes"/>
 <layer number="91" name="Nets" color="2" fill="1" visible="yes" active="yes"/>
@@
 <layer number="97" name="Info" color="7" fill="1" visible="yes" active="yes"/>
 <layer number="98" name="Guide" color="6" fill="1" visible="yes" active="yes"/>
+<layer number="100" name="Muster" color="7" fill="1" visible="no" active="no"/>
+<layer number="101" name="Patch_Top" color="12" fill="4" visible="yes" active="yes"/>
+<layer number="102" name="Vscore" color="7" fill="1" visible="yes" active="yes"/>
+<layer number="103" name="tMap" color="7" fill="1" visible="yes" active="yes"/>
+<layer number="104" name="Name" color="16" fill="1" visible="yes" active="yes"/>
+<layer number="105" name="Beschreib" color="9" fill="1" visible="no" active="no"/>
+<layer number="106" name="BGA-Top" color="4" fill="1" visible="no" active="no"/>
+<layer number="107" name="BD-Top" color="5" fill="1" visible="no" active="no"/>
+<layer number="116" name="Patch_BOT" color="9" fill="4" visible="yes" active="yes"/>
+<layer number="121" name="_tsilk" color="7" fill="1" visible="yes" active="yes"/>
+<layer number="122" name="_bsilk" color="7" fill="1" visible="yes" active="yes"/>
+<layer number="125" name="_tNames" color="7" fill="1" visible="yes" active="yes"/>
+<layer number="144" name="Drill_legend" color="7" fill="1" visible="yes" active="yes"/>
+<layer number="151" name="HeatSink" color="7" fill="1" visible="yes" active="yes"/>
+<layer number="200" name="200bmp" color="1" fill="10" visible="no" active="no"/>
+<layer number="201" name="201bmp" color="2" fill="10" visible="yes" active="yes"/>
+<layer number="202" name="202bmp" color="3" fill="10" visible="yes" active="yes"/>
+<layer number="203" name="203bmp" color="4" fill="10" visible="yes" active="yes"/>
+<layer number="204" name="204bmp" color="5" fill="10" visible="yes" active="yes"/>
+<layer number="205" name="205bmp" color="6" fill="10" visible="yes" active="yes"/>
+<layer number="206" name="206bmp" color="7" fill="10" visible="yes" active="yes"/>
+<layer number="207" name="207bmp" color="8" fill="10" visible="yes" active="yes"/>
+<layer number="208" name="208bmp" color="9" fill="10" visible="yes" active="yes"/>
+<layer number="209" name="209bmp" color="7" fill="1" visible="yes" active="yes"/>
+<layer number="210" name="210bmp" color="7" fill="1" visible="yes" active="yes"/>
+<layer number="211" name="211bmp" color="7" fill="1" visible="yes" active="yes"/>
+<layer number="212" name="212bmp" color="7" fill="1" visible="yes" active="yes"/>
+<layer number="213" name="213bmp" color="7" fill="1" visible="yes" active="yes"/>
+<layer number="214" name="214bmp" color="7" fill="1" visible="yes" active="yes"/>
+<layer number="215" name="215bmp" color="7" fill="1" visible="yes" active="yes"/>
+<layer number="216" name="216bmp" color="7" fill="1" visible="yes" active="yes"/>
+<layer number="231" name="Eagle3D_PG1" color="14" fill="1" visible="yes" active="yes"/>
+<layer number="232" name="Eagle3D_PG2" color="14" fill="2" visible="yes" active="yes"/>
+<layer number="233" name="Eagle3D_PG3" color="14" fill="4" visible="yes" active="yes"/>
+<layer number="250" name="Descript" color="3" fill="1" visible="no" active="no"/>
+<layer number="251" name="SMDround" color="12" fill="11" visible="no" active="no"/>
+<layer number="254" name="cooling" color="7" fill="1" visible="yes" active="yes"/>
 </layers>
 <schematic xreflabel="%F%N/%S.%C%R" xrefpart="/%S.%C%R">
@@
 <parts>
 <part name="IC1" library="xmega-a4" deviceset="AT-XMEGA-XXA4-AU" device=""/>
+<part name="U$1" library="SHC" deviceset="MS5611" device="QFN"/>
+<part name="U$2" library="SHC" deviceset="M10382-A1" device=""/>
+<part name="U$3" library="SHC" deviceset="123_BATTERY_HOLDER" device="CR-123-A"/>
+<part name="U$4" library="SHC" deviceset="123_BATTERY_HOLDER" device="CR-123-A"/>
+<part name="U$5" library="SHC" deviceset="123_BATTERY_HOLDER" device="CR-123-A"/>
+<part name="U$6" library="SHC" deviceset="123_BATTERY_HOLDER" device="CR-123-A"/>
+<part name="U$7" library="SHC" deviceset="123_BATTERY_HOLDER" device="CR-123-A"/>
+<part name="U$8" library="SHC" deviceset="123_BATTERY_HOLDER" device="CR-123-A"/>
 </parts>
 <sheets>
@@
 <instances>
 <instance part="IC1" gate="G$1" x="78.74" y="66.04"/>
+<instance part="U$1" gate="G$1" x="22.86" y="121.92"/>
+<instance part="U$2" gate="G$1" x="17.78" y="78.74"/>
+<instance part="U$3" gate="G$1" x="10.16" y="40.64"/>
+<instance part="U$4" gate="G$1" x="20.32" y="40.64"/>
+<instance part="U$5" gate="G$1" x="30.48" y="40.64"/>
+<instance part="U$6" gate="G$1" x="10.16" y="27.94"/>
+<instance part="U$7" gate="G$1" x="20.32" y="27.94"/>
+<instance part="U$8" gate="G$1" x="30.48" y="27.94"/>
 </instances>
 <busses>

Commit message: April 8th work.
Parts:
- added C1, C2, C3, C5: 22pF, SparkFun:CAP0805
- added C6: 18pF, SparkFun:CAP0805
- added C7: 100nF, SparkFun:CAP0805
- added IC2, IC3: 74AHC1G125DBV, 74xx-little-us:74AHC1G125DBV
- added JP1, JP2, JP3: (no value), SparkFun-Connectors:M03JST-PTH
- added L3, L4: FB_0402, rc-master-smd:FB_0402
- added M1: HX1, trackuino:HX1
- added MPU: (no value), con-amp-quick:M04
- added U$9: AVR-PDIVERT, avr-7:AVR-PDIVERT
- added X1: BU-SMA-V, con-coax:BU-SMA-V
Connections:
- new net 5V: IC2P.VCC, IC3P.VCC, M1.VCC
- new net BATT: JP1.2, JP2.2, U$5.+, U$8.+
- new net EN-5V: IC3A.O, M1.EN
- new net GC1: IC1.PA2/ADC2, JP1.3
- new net GC2: IC1.PA3/ADC3, JP2.3
- new net GND: C1.2, C2.2, C3.2, C5.2, C6.1, C6.2, C7.2, IC1.GND@1, IC1.GND@2, IC1.GND@3, IC1.GND@4, IC2A.OE, IC2P.GND, IC3A.OE, IC3P.GND, JP1.1, JP2.1, JP3.1, M1.0V, M1.BODYGND1, M1.BODYGND2, M1.RFGND1, M1.RFGND2, MPU.4, U$1.!CS!, U$1.GND, U$1.PS, U$2.ANT_IN, U$2.ANT_OUT, U$2.GND, U$2.V_TH, U$3.-, U$6.-, U$9.6, X1G$1.GND
- new net MISOC: IC1.PC6/MISO/RXD1, U$1.MISO
- new net MOSIC: IC1.PC5/OC1B/MOSI/XCK1, U$1.MOSI/SDA
- new net N$1: C1.1, L3.2, U$2.TX
- new net N$2: C2.1, L4.2, U$2.RX
- new net N$4: U$3.+, U$4.-
- new net N$5: M1.RFOUT, X1G$1.1
- new net N$6: U$4.+, U$5.-
- new net N$8: U$6.+, U$7.-
- new net N$9: U$7.+, U$8.-
- new net PDI-CLK: IC1.RESET/PDI-CLK, U$9.5
- new net PDI-DATA: IC1.PDI-DATA, U$9.1
- new net RXC: IC1.PC2/OC0C/RXD0, L3.1
- new net RXE: IC1.!!RXD0OC0CPE2, IC2A.I
- new net SCLKC: IC1.PC7/SCK/TXD1/CLKO/EVO, U$1.SCLK
- new net SCLKD: IC1.!!!TXD1SCKCLKOPD7, MPU.1
- new net SDID: IC1.!!XCK1MOSIPD5, MPU.2
- new net THERM: IC1.PA1/ADC1, JP3.3
- new net TXC: IC1.PC3/OC0D/TXD0, L4.1
- new net TXD-5V: IC2A.O, M1.TXD
- new net TXE: IC1.!!TXD0OC0DPE3, IC3A.I
- new net VCC: C3.1, C5.1, C7.1, IC1.VCC@1, IC1.VCC@2, IC1.VCC@3, JP3.2, MPU.3, U$1.VDD, U$2.VCC, U$2.VIO, U$9.2
Other:
- moved on the sheet: U$1, U$2

Commit message: New Volt Reg Lib
Parts:
- added U$10: AZ1117EH-3.33.3, Physoon:AZ1117EH-3.33.3
Changed lines of the file:
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@@
 <?xml version="1.0" encoding="utf-8"?>
 <!DOCTYPE eagle SYSTEM "eagle.dtd">
-<eagle version="6.5.0">
+<eagle version="8.1.0">
 <drawing>
 <settings>
@@
 <setting verticaltext="up"/>
 </settings>
-<grid distance="0.1" unitdist="inch" unit="inch" style="lines" multiple="1" display="yes" altdistance="0.01" altunitdist="inch" altunit="inch"/>
+<grid distance="0.1" unitdist="inch" unit="inch" style="lines" multiple="1" display="no" altdistance="0.01" altunitdist="inch" altunit="inch"/>
 <layers>
-<layer number="1" name="Top" color="4" fill="1" visible="yes" active="no"/>
-<layer number="16" name="Bottom" color="1" fill="1" visible="yes" active="no"/>
-<layer number="17" name="Pads" color="2" fill="1" visible="yes" active="no"/>
-<layer number="18" name="Vias" color="2" fill="1" visible="yes" active="no"/>
-<layer number="19" name="Unrouted" color="6" fill="1" visible="yes" active="no"/>
-<layer number="20" name="Dimension" color="15" fill="1" visible="yes" active="no"/>
-<layer number="21" name="tPlace" color="7" fill="1" visible="yes" active="no"/>
-<layer number="22" name="bPlace" color="7" fill="1" visible="yes" active="no"/>
-<layer number="23" name="tOrigins" color="15" fill="1" visible="yes" active="no"/>
-<layer number="24" name="bOrigins" color="15" fill="1" visible="yes" active="no"/>
-<layer number="25" name="tNames" color="7" fill="1" visible="yes" active="no"/>
-<layer number="26" name="bNames" color="7" fill="1" visible="yes" active="no"/>
-<layer number="27" name="tValues" color="7" fill="1" visible="yes" active="no"/>
-<layer number="28" name="bValues" color="7" fill="1" visible="yes" active="no"/>
+<layer number="1" name="Top" color="4" fill="1" visible="no" active="no"/>
+<layer number="16" name="Bottom" color="1" fill="1" visible="no" active="no"/>
+<layer number="17" name="Pads" color="2" fill="1" visible="no" active="no"/>
+<layer number="18" name="Vias" color="2" fill="1" visible="no" active="no"/>
+<layer number="19" name="Unrouted" color="6" fill="1" visible="no" active="no"/>
+<layer number="20" name="Dimension" color="15" fill="1" visible="no" active="no"/>
+<layer number="21" name="tPlace" color="7" fill="1" visible="no" active="no"/>
+<layer number="22" name="bPlace" color="7" fill="1" visible="no" active="no"/>
+<layer number="23" name="tOrigins" color="15" fill="1" visible="no" active="no"/>
+<layer number="24" name="bOrigins" color="15" fill="1" visible="no" active="no"/>
+<layer number="25" name="tNames" color="7" fill="1" visible="no" active="no"/>
+<layer number="26" name="bNames" color="7" fill="1" visible="no" active="no"/>
+<layer number="27" name="tValues" color="7" fill="1" visible="no" active="no"/>
+<layer number="28" name="bValues" color="7" fill="1" visible="no" active="no"/>
 <layer number="29" name="tStop" color="7" fill="3" visible="no" active="no"/>
 <layer number="30" name="bStop" color="7" fill="6" visible="no" active="no"/>
@@
 <layer number="35" name="tGlue" color="7" fill="4" visible="no" active="no"/>
 <layer number="36" name="bGlue" color="7" fill="5" visible="no" active="no"/>
-<layer number="37" name="tTest" color="7" fill="1" visible="yes" active="no"/>
-<layer number="38" name="bTest" color="7" fill="1" visible="yes" active="no"/>
+<layer number="37" name="tTest" color="7" fill="1" visible="no" active="no"/>
+<layer number="38" name="bTest" color="7" fill="1" visible="no" active="no"/>
 <layer number="39" name="tKeepout" color="4" fill="11" visible="no" active="no"/>
 <layer number="40" name="bKeepout" color="1" fill="11" visible="no" active="no"/>
@@
 <layer number="44" name="Drills" color="7" fill="1" visible="no" active="no"/>
 <layer number="45" name="Holes" color="7" fill="1" visible="no" active="no"/>
-<layer number="46" name="Milling" color="3" fill="1" visible="yes" active="no"/>
-<layer number="47" name="Measures" color="7" fill="1" visible="yes" active="no"/>
-<layer number="48" name="Document" color="7" fill="1" visible="yes" active="no"/>
-<layer number="49" name="Reference" color="7" fill="1" visible="yes" active="no"/>
-<layer number="50" name="dxf" color="7" fill="1" visible="yes" active="no"/>
-<layer number="51" name="tDocu" color="7" fill="1" visible="yes" active="no"/>
-<layer number="52" name="bDocu" color="7" fill="1" visible="yes" active="no"/>
-<layer number="53" name="tGND_GNDA" color="7" fill="9" visible="yes" active="no"/>
-<layer number="54" name="bGND_GNDA" color="1" fill="9" visible="yes" active="no"/>
-<layer number="56" name="wert" color="7" fill="1" visible="yes" active="no"/>
-<layer number="60" name="p_dimension" color="7" fill="1" visible="yes" active="no"/>
-<layer number="61" name="pt_docu" color="7" fill="1" visible="yes" active="no"/>
+<layer number="46" name="Milling" color="3" fill="1" visible="no" active="no"/>
+<layer number="47" name="Measures" color="7" fill="1" visible="no" active="no"/>
+<layer number="48" name="Document" color="7" fill="1" visible="no" active="no"/>
+<layer number="49" name="Reference" color="7" fill="1" visible="no" active="no"/>
+<layer number="50" name="dxf" color="7" fill="1" visible="no" active="no"/>
+<layer number="51" name="tDocu" color="7" fill="1" visible="no" active="no"/>
+<layer number="52" name="bDocu" color="7" fill="1" visible="no" active="no"/>
+<layer number="53" name="tGND_GNDA" color="7" fill="9" visible="no" active="no"/>
+<layer number="54" name="bGND_GNDA" color="1" fill="9" visible="no" active="no"/>
+<layer number="56" name="wert" color="7" fill="1" visible="no" active="no"/>
+<layer number="60" name="p_dimension" color="7" fill="1" visible="no" active="no"/>
+<layer number="61" name="pt_docu" color="7" fill="1" visible="no" active="no"/>
 <layer number="90" name="Modules" color="5" fill="1" visible="yes" active="yes"/>
 <layer number="91" name="Nets" color="2" fill="1" visible="yes" active="yes"/>
@@
 <part name="GND23" library="SparkFun-Aesthetics" deviceset="GND" device=""/>
 <part name="GND24" library="SparkFun-Aesthetics" deviceset="GND" device=""/>
+<part name="U$10" library="Physoon" deviceset="AZ1117EH-3.3" device="3.3"/>
 </parts>
 <sheets>
@@
 <instance part="GND23" gate="1" x="2.54" y="66.04"/>
 <instance part="GND24" gate="1" x="-78.74" y="-29.21" rot="R270"/>
+<instance part="U$10" gate="G$1" x="71.12" y="185.42"/>
 </instances>
 <busses>
