File: Main.brd (EAGLE design)
At the start: 100 x 80 mm, 34 parts, among them IC2 74AHC1G125DBV, IC3 74AHC1G125DBV, M1 HX1, X1 BU-SMA-V

Commit message: idk
Parts:
- moved U$6 5.00 mm to (72.5, 10.2)
- moved U$3 4.60 mm to (27.5, 10.2)
Routing:
- net GND: track 459.6 -> 454.3 mm
- net N$8: track 19.1 -> 19.7 mm
- net N$4: track 19.1 -> 19.6 mm
Changed lines of the file:
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@@
 <?xml version="1.0" encoding="utf-8"?>
 <!DOCTYPE eagle SYSTEM "eagle.dtd">
-<eagle version="8.1.0">
+<eagle version="6.5.0">
 <drawing>
 <settings>
@@
 <setting verticaltext="up"/>
 </settings>
-<grid distance="1" unitdist="mm" unit="mm" style="lines" multiple="1" display="yes" altdistance="0.1" altunitdist="mm" altunit="mm"/>
+<grid distance="0.0393700787" unitdist="inch" unit="inch" style="lines" multiple="1" display="yes" altdistance="3.93700787" altunitdist="mil" altunit="inch"/>
 <layers>
 <layer number="1" name="Top" color="4" fill="1" visible="yes" active="yes"/>
@@
 <layer number="20" name="Dimension" color="15" fill="1" visible="yes" active="yes"/>
 <layer number="21" name="tPlace" color="7" fill="1" visible="yes" active="yes"/>
-<layer number="22" name="bPlace" color="7" fill="1" visible="yes" active="yes"/>
+<layer number="22" name="bPlace" color="7" fill="1" visible="no" active="yes"/>
 <layer number="23" name="tOrigins" color="15" fill="1" visible="no" active="yes"/>
 <layer number="24" name="bOrigins" color="15" fill="1" visible="no" active="yes"/>
-<layer number="25" name="tNames" color="7" fill="1" visible="no" active="yes"/>
-<layer number="26" name="bNames" color="7" fill="1" visible="no" active="yes"/>
+<layer number="25" name="tNames" color="7" fill="1" visible="yes" active="yes"/>
+<layer number="26" name="bNames" color="7" fill="1" visible="yes" active="yes"/>
 <layer number="27" name="tValues" color="7" fill="1" visible="no" active="yes"/>
 <layer number="28" name="bValues" color="7" fill="1" visible="no" active="yes"/>
@@
 <layer number="43" name="vRestrict" color="2" fill="10" visible="no" active="yes"/>
 <layer number="44" name="Drills" color="7" fill="1" visible="no" active="yes"/>
-<layer number="45" name="Holes" color="7" fill="1" visible="no" active="yes"/>
+<layer number="45" name="Holes" color="7" fill="1" visible="yes" active="yes"/>
 <layer number="46" name="Milling" color="3" fill="1" visible="no" active="yes"/>
 <layer number="47" name="Measures" color="7" fill="1" visible="no" active="yes"/>
@@
 <layer number="49" name="Reference" color="7" fill="1" visible="no" active="yes"/>
 <layer number="50" name="dxf" color="7" fill="1" visible="no" active="no"/>
-<layer number="51" name="tDocu" color="7" fill="1" visible="no" active="yes"/>
-<layer number="52" name="bDocu" color="7" fill="1" visible="no" active="yes"/>
+<layer number="51" name="tDocu" color="7" fill="1" visible="yes" active="yes"/>
+<layer number="52" name="bDocu" color="7" fill="1" visible="yes" active="yes"/>
 <layer number="53" name="tGND_GNDA" color="7" fill="9" visible="no" active="no"/>
 <layer number="54" name="bGND_GNDA" color="1" fill="9" visible="no" active="no"/>
@@
 <wire x1="100" y1="80" x2="0" y2="80" width="0" layer="20"/>
 <wire x1="0" y1="80" x2="0" y2="0" width="0" layer="20"/>
-<text x="55" y="1" size="2.54" layer="21" rot="R90">Physoon 2.0</text>
+<text x="55" y="20" size="2.54" layer="21" rot="R90">Physoon 2.0</text>
 <text x="27" y="18" size="2.54" layer="22" rot="MR0">GPS</text>
 <text x="12" y="52" size="1.778" layer="22" rot="MR0">MS5607</text>
@@
 <text x="86" y="59" size="1.27" layer="22" rot="MR0">LOGIC</text>
 <text x="6" y="21" size="1.27" layer="22" rot="MR0">18pF</text>
-<text x="6" y="6" size="1.27" layer="22" rot="MR0">GND</text>
+<text x="11" y="6" size="1.27" layer="22" rot="MR0">GND</text>
 <text x="60.3" y="6" size="1.27" layer="22" rot="MR0">GND</text>
-<text x="2" y="6" size="1.27" layer="21">GND</text>
+<text x="7" y="6" size="1.27" layer="21">GND</text>
 <text x="56.3" y="6" size="1.27" layer="21">GND</text>
 <text x="94" y="45" size="1.27" layer="21">BATT</text>
@@
 <rectangle x1="74.8919" y1="31.1531" x2="75.0189" y2="31.1785" layer="22"/>
 <text x="0" y="-0.127" size="0.0508" layer="209" font="vector">/storage/Chrome/croc.bmp</text>
+<hole x="3" y="4" drill="2.2606"/>
+<hole x="97" y="4" drill="2.2606"/>
+<hole x="3" y="77.5" drill="2.2606"/>
+<hole x="50" y="40" drill="2"/>
 </plain>
 <attributes>
@@
 <pass name="Default">
 <param name="RoutingGrid" value="50mil"/>
-<param name="AutoGrid" value="1"/>
-<param name="Efforts" value="0"/>
-<param name="TopRouterVariant" value="1"/>
 <param name="tpViaShape" value="round"/>
 <param name="PrefDir.1" value="|"/>
@@
 <element name="U$1" library="SHC" package="MS5611-01BA01" value="MS5611QFN" x="8.89" y="46.99" rot="MR180"/>
 <element name="U$2" library="SHC" package="M10382-A1" value="M10382-A1" x="22.86" y="19.05" rot="MR270"/>
-<element name="U$3" library="SHC" package="CR-123-A_HOLDER" value="123_BATTERY_HOLDERCR-123-A" x="22.86" y="10.16" rot="R180"/>
+<element name="U$3" library="SHC" package="CR-123-A_HOLDER" value="123_BATTERY_HOLDERCR-123-A" x="27.46" y="10.16" rot="R180"/>
 <element name="U$4" library="SHC" package="CR-123-A_HOLDER" value="123_BATTERY_HOLDERCR-123-A" x="22.86" y="29.21"/>
 <element name="U$5" library="SHC" package="CR-123-A_HOLDER" value="123_BATTERY_HOLDERCR-123-A" x="22.86" y="48.26" rot="R180"/>
-<element name="U$6" library="SHC" package="CR-123-A_HOLDER" value="123_BATTERY_HOLDERCR-123-A" x="77.47" y="10.16" rot="R180"/>
+<element name="U$6" library="SHC" package="CR-123-A_HOLDER" value="123_BATTERY_HOLDERCR-123-A" x="72.47" y="10.16" rot="R180"/>
 <element name="U$7" library="SHC" package="CR-123-A_HOLDER" value="123_BATTERY_HOLDERCR-123-A" x="77.47" y="29.21"/>
 <element name="U$8" library="SHC" package="CR-123-A_HOLDER" value="123_BATTERY_HOLDERCR-123-A" x="77.47" y="48.26" rot="R180"/>
@@
 <wire x1="10.76" y1="16.4" x2="10.76" y2="14.8" width="0.4064" layer="16"/>
 <wire x1="10.76" y1="14.8" x2="8.45" y2="14.8" width="0.4064" layer="16"/>
-<wire x1="8.45" y1="14.8" x2="3.81" y2="10.16" width="0.4064" layer="16"/>
+<wire x1="8.45" y1="14.8" x2="8.41" y2="10.16" width="0.4064" layer="16"/>
 <wire x1="10.76" y1="14.8" x2="12.76" y2="14.8" width="0.4064" layer="16"/>
 <wire x1="12.76" y1="14.8" x2="13.26" y2="14.3" width="0.4064" layer="16"/>
@@
 <wire x1="34.06" y1="13.105" x2="34.06" y2="7.85" width="0.4064" layer="16"/>
 <wire x1="34.06" y1="7.85" x2="34.29" y2="7.62" width="0.4064" layer="16"/>
-<wire x1="34.29" y1="7.62" x2="55.88" y2="7.62" width="0.4064" layer="16"/>
-<wire x1="55.88" y1="7.62" x2="58.42" y2="10.16" width="0.4064" layer="16"/>
 <wire x1="29.26" y1="23.8" x2="29.21" y2="23.85" width="0.4064" layer="16"/>
 <wire x1="26.035" y1="23.825" x2="26.06" y2="23.8" width="0.4064" layer="16"/>
@@
 <wire x1="33.655" y1="22.225" x2="34.06" y2="23.8" width="0.4064" layer="16"/>
 <wire x1="28.575" y1="22.225" x2="33.655" y2="22.225" width="0.4064" layer="16"/>
-<wire x1="22.595" y1="26.035" x2="20.13393125" y2="27.657821875" width="0.4064" layer="16"/>
-<wire x1="20.13393125" y1="27.657821875" x2="17.78" y2="29.21" width="0.4064" layer="16"/>
+<wire x1="22.595" y1="26.035" x2="21.13393125" y2="27.657821875" width="0.4064" layer="16"/>
+<wire x1="21.13393125" y1="27.657821875" x2="17.78" y2="29.21" width="0.4064" layer="16"/>
 <wire x1="17.78" y1="29.21" x2="13.335" y2="29.21" width="0.4064" layer="16"/>
 <wire x1="13.335" y1="29.21" x2="13.07" y2="26.67" width="0.4064" layer="16"/>
 <wire x1="29.475" y1="26.035" x2="29.26" y2="23.8" width="0.4064" layer="16"/>
-<wire x1="19.99" y1="42.51" x2="20.13393125" y2="27.657821875" width="0.4064" layer="16"/>
+<wire x1="19.99" y1="42.51" x2="21.13393125" y2="27.657821875" width="0.4064" layer="16"/>
 <wire x1="13.26" y1="23.8" x2="12.59" y2="21.7" width="0.4064" layer="16"/>
 <wire x1="10.16" y1="69.85" x2="10.16" y2="66.675" width="0.4064" layer="1"/>
@@
 <vertex x="0" y="0"/>
 </polygon>
+<wire x1="34.29" y1="7.62" x2="53.42" y2="7.62" width="0.4064" layer="16"/>
+<wire x1="53.42" y1="7.62" x2="53.42" y2="10.16" width="0.4064" layer="16"/>
 </signal>
 <signal name="PDI-DATA">
@@
 <contactref element="U$3" pad="+"/>
 <contactref element="U$4" pad="-"/>
-<wire x1="41.91" y1="10.16" x2="41.91" y2="29.21" width="0.4064" layer="16"/>
+<wire x1="46.51" y1="10.16" x2="41.91" y2="29.21" width="0.4064" layer="16"/>
 </signal>
 <signal name="N$6">
@@
 <contactref element="U$6" pad="+"/>
 <contactref element="U$7" pad="-"/>
-<wire x1="96.52" y1="29.21" x2="96.52" y2="10.16" width="0.4064" layer="16"/>
+<wire x1="96.52" y1="29.21" x2="91.52" y2="10.16" width="0.4064" layer="16"/>
 </signal>
 <signal name="N$9">
