File: Main.brd (EAGLE design)
At the start: 100 x 80 mm, 34 parts, among them IC2 74AHC1G125DBV, IC3 74AHC1G125DBV, M1 HX1, X1 BU-SMA-V

Commit message: Add LED for nerde programmers
Parts:
- added LED1: (no value), led:CHIP-LED0603
- added R1: 220, rcl:R0603
Connections:
- new net LED: IC1.1, R1.1
- new net N$11: LED1.A, R1.2
- net GND: now also LED1.C
Routing:
- net LED: track 0.00 -> 25.8 mm, vias 0 -> 1
- net GND: track 453.9 -> 479.5 mm
- net N$11: track 0.00 -> 3.04 mm
Changed lines of the file:
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@@
 <layer number="21" name="tPlace" color="7" fill="1" visible="yes" active="yes"/>
 <layer number="22" name="bPlace" color="7" fill="1" visible="yes" active="yes"/>
-<layer number="23" name="tOrigins" color="15" fill="1" visible="no" active="yes"/>
-<layer number="24" name="bOrigins" color="15" fill="1" visible="no" active="yes"/>
+<layer number="23" name="tOrigins" color="15" fill="1" visible="yes" active="yes"/>
+<layer number="24" name="bOrigins" color="15" fill="1" visible="yes" active="yes"/>
 <layer number="25" name="tNames" color="7" fill="1" visible="no" active="yes"/>
 <layer number="26" name="bNames" color="7" fill="1" visible="no" active="yes"/>
@@
 <element name="JP4" library="SparkFun" package="MOLEX-1X6" value="" x="15.24" y="69.85"/>
 <element name="U$12" library="SHC" package="ZMCHFL3R" value="CKN10160-ND" x="38.1" y="76.2"/>
+<element name="LED1" library="led" package="CHIP-LED0603" value="" x="50" y="34" rot="R90"/>
+<element name="R1" library="rcl" package="R0603" value="220" x="50" y="37"/>
 </elements>
 <signals>
@@
 <wire x1="82.6" y1="63.2" x2="82.42236875" y2="63.2" width="0.4064" layer="16"/>
 <wire x1="82.42236875" y1="63.2" x2="82.42236875" y2="61.52236875" width="0.4064" layer="16"/>
+<contactref element="LED1" pad="C"/>
+<wire x1="49.25" y1="34" x2="49.25" y2="14.33" width="0.4064" layer="1"/>
+<wire x1="49.25" y1="14.33" x2="53.42" y2="10.16" width="0.4064" layer="1"/>
 </signal>
 <signal name="PDI-DATA">
@@
 <wire x1="56.74210625" y1="62.865" x2="56.13250625" y2="63.4746" width="0.4064" layer="16"/>
 </signal>
+<signal name="N$11">
+<contactref element="R1" pad="2"/>
+<contactref element="LED1" pad="A"/>
+<wire x1="50.75" y1="34" x2="50.75" y2="36.9" width="0.4064" layer="1"/>
+<wire x1="50.75" y1="36.9" x2="50.85" y2="37" width="0.4064" layer="1"/>
+</signal>
+<signal name="LED">
+<contactref element="IC1" pad="1"/>
+<contactref element="R1" pad="1"/>
+<wire x1="49.15" y1="37" x2="48" y2="37" width="0.4064" layer="1"/>
+<wire x1="48" y1="37" x2="47" y2="38" width="0.4064" layer="1"/>
+<via x="47" y="38" extent="1-16" drill="0.6"/>
+<wire x1="47" y1="38" x2="30.1" y2="38" width="0.4064" layer="16"/>
+<wire x1="30.1" y1="38" x2="25.59" y2="42.51" width="0.4064" layer="16"/>
+</signal>
 </signals>
