File: RemovingGround.brd (EAGLE design)
At the start: 100 x 80 mm, 34 parts, among them IC2 74AHC1G125DBV, IC3 74AHC1G125DBV, M1 HX1, X1 BU-SMA-V

Commit message: gf
Parts:
- added LED1: (no value), led:CHIP-LED0603
- added R1: 220, resistor:R0603
Connections:
- new net LED: IC1.1, R1.1
- new net N$10: LED1.A, R1.2
- net GND: now also LED1.C
Routing:
- net LED: track 0.00 -> 26.9 mm, vias 0 -> 1
- net N$10: track 0.00 -> 3.10 mm
Changed lines of the file:
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@@
 <?xml version="1.0" encoding="utf-8"?>
 <!DOCTYPE eagle SYSTEM "eagle.dtd">
-<eagle version="8.1.0">
+<eagle version="6.5.0">
 <drawing>
 <settings>
@@
 <pass name="Default">
 <param name="RoutingGrid" value="50mil"/>
-<param name="AutoGrid" value="1"/>
-<param name="Efforts" value="0"/>
-<param name="TopRouterVariant" value="1"/>
 <param name="tpViaShape" value="round"/>
 <param name="PrefDir.1" value="|"/>
@@
 <element name="JP4" library="SparkFun" package="MOLEX-1X6" value="" x="15.24" y="69.85"/>
 <element name="U$12" library="SHC" package="ZMCHFL3R" value="CKN10160-ND" x="38.1" y="76.2"/>
+<element name="LED1" library="led" package="CHIP-LED0603" value="" x="49" y="29" rot="R90"/>
+<element name="R1" library="resistor" package="R0603" value="220" x="49" y="32"/>
 </elements>
 <signals>
@@
 <wire x1="20.1504" y1="45" x2="18" y2="45" width="0.4064" layer="1"/>
 <via x="18" y="45" extent="1-16" drill="0.6"/>
+<contactref element="LED1" pad="C"/>
+<wire x1="97.7999" y1="69.8401" x2="97.7999" y2="74.9399" width="0" layer="19" extent="1-1"/>
+<wire x1="92.7001" y1="74.9399" x2="97.7999" y2="74.9399" width="0" layer="19" extent="1-1"/>
+<wire x1="92.7001" y1="69.8401" x2="97.7999" y2="69.8401" width="0" layer="19" extent="1-1"/>
+<wire x1="86.995" y1="78.105" x2="92.7001" y2="74.9399" width="0" layer="19" extent="1-1"/>
+<wire x1="83.84" y1="63.18" x2="92.7001" y2="69.8401" width="0" layer="19" extent="16-16"/>
+<wire x1="83.84" y1="61.28" x2="83.84" y2="63.18" width="0" layer="19" extent="16-16"/>
+<wire x1="76.2" y1="60.96" x2="83.84" y2="61.28" width="0" layer="19" extent="16-16"/>
+<wire x1="66.02" y1="60.64" x2="76.2" y2="60.96" width="0" layer="19" extent="16-16"/>
+<wire x1="66.2186" y1="58.9386" x2="66.02" y2="60.64" width="0" layer="19" extent="16-16"/>
+<wire x1="55.88" y1="60.96" x2="66.02" y2="60.64" width="0" layer="19" extent="16-16"/>
+<wire x1="50.8" y1="60.96" x2="55.88" y2="60.96" width="0" layer="19" extent="1-1"/>
+<wire x1="43.91" y1="64.69" x2="50.8" y2="60.96" width="0" layer="19" extent="1-1"/>
+<wire x1="35.02" y1="64.69" x2="43.91" y2="64.69" width="0" layer="19" extent="1-1"/>
+<wire x1="26.13" y1="64.69" x2="35.02" y2="64.69" width="0" layer="19" extent="1-1"/>
+<wire x1="25.4" y1="69.85" x2="26.13" y2="64.69" width="0" layer="19" extent="1-1"/>
+<wire x1="63.285" y1="48.895" x2="66.02" y2="58.74" width="0" layer="19" extent="16-16"/>
+<wire x1="63.5" y1="46.57" x2="63.5" y2="48.68" width="0" layer="19" extent="16-16"/>
+<wire x1="67.14" y1="48.26" x2="63.5" y2="48.68" width="0" layer="19" extent="16-16"/>
+<wire x1="63.5" y1="41.06" x2="63.5" y2="46.57" width="0" layer="19" extent="16-16"/>
+<wire x1="63.5" y1="37.25" x2="63.5" y2="41.06" width="0" layer="19" extent="16-16"/>
+<wire x1="67.14" y1="37.07" x2="63.5" y2="37.25" width="0" layer="19" extent="16-16"/>
+<wire x1="73.34" y1="48.26" x2="67.14" y2="48.26" width="0" layer="19" extent="16-16"/>
+<wire x1="23.19" y1="54.01" x2="26.13" y2="64.69" width="0" layer="19" extent="16-16"/>
+<wire x1="27.34" y1="49.06" x2="23.19" y2="54.01" width="0" layer="19" extent="16-16"/>
+<wire x1="20.1504" y1="45" x2="27.34" y2="49.06" width="0" layer="19" extent="1-16"/>
+<wire x1="15.84" y1="49.06" x2="18" y2="45" width="0" layer="19" extent="16-16"/>
+<wire x1="7.69" y1="46.365" x2="7.69" y2="47.615" width="0" layer="19" extent="16-16"/>
+<wire x1="3.815" y1="44.72" x2="6" y2="47.615" width="0" layer="19" extent="16-16"/>
+<wire x1="48.895" y1="78.105" x2="43.91" y2="64.69" width="0" layer="19" extent="1-1"/>
+<wire x1="5.08" y1="64.77" x2="6" y2="50" width="0" layer="19" extent="16-16"/>
+<wire x1="10.16" y1="69.85" x2="5.08" y2="64.77" width="0" layer="19" extent="1-1"/>
+<wire x1="22.595" y1="26.035" x2="19.99" y2="42.51" width="0" layer="19" extent="16-16"/>
+<wire x1="26.035" y1="23.825" x2="22.595" y2="26.035" width="0" layer="19" extent="16-16"/>
+<wire x1="29.21" y1="23.85" x2="26.06" y2="23.8" width="0" layer="19" extent="16-16"/>
+<wire x1="29.475" y1="26.035" x2="29.21" y2="23.85" width="0" layer="19" extent="16-16"/>
+<wire x1="34.06" y1="23.8" x2="29.26" y2="23.8" width="0" layer="19" extent="16-16"/>
+<wire x1="29.26" y1="14.3" x2="29.21" y2="23.75" width="0" layer="19" extent="16-16"/>
+<wire x1="26.3" y1="14.06" x2="29.26" y2="14.3" width="0" layer="19" extent="16-16"/>
+<wire x1="26.3" y1="11.43" x2="26.3" y2="14.06" width="0" layer="19" extent="16-16"/>
+<wire x1="22.86" y1="14.3" x2="26.06" y2="14.3" width="0" layer="19" extent="16-16"/>
+<wire x1="34.06" y1="14.3" x2="29.26" y2="14.3" width="0" layer="19" extent="16-16"/>
+<wire x1="14.86" y1="14.3" x2="22.86" y2="14.3" width="0" layer="19" extent="16-16"/>
+<wire x1="13.26" y1="14.3" x2="14.86" y2="14.3" width="0" layer="19" extent="16-16"/>
+<wire x1="10.76" y1="14.8" x2="13.26" y2="14.3" width="0" layer="19" extent="16-16"/>
+<wire x1="10.76" y1="16.4" x2="10.76" y2="14.8" width="0" layer="19" extent="16-16"/>
+<wire x1="10.76" y1="20.1" x2="10.795" y2="16.435" width="0" layer="19" extent="16-16"/>
+<wire x1="10.65" y1="21.59" x2="10.76" y2="20.1" width="0" layer="19" extent="16-16"/>
+<wire x1="10.76" y1="23.3" x2="10.76" y2="21.7" width="0" layer="19" extent="16-16"/>
+<wire x1="13.07" y1="23.99" x2="10.76" y2="23.3" width="0" layer="19" extent="16-16"/>
+<wire x1="13.07" y1="26.67" x2="13.07" y2="23.99" width="0" layer="19" extent="16-16"/>
+<wire x1="7.99" y1="20.69" x2="10.65" y2="21.59" width="0" layer="19" extent="16-16"/>
+<wire x1="7.62" y1="22.49" x2="7.62" y2="20.69" width="0" layer="19" extent="16-16"/>
+<wire x1="8.41" y1="10.16" x2="10.76" y2="14.8" width="0" layer="19" extent="16-16"/>
+<wire x1="48.25" y1="29" x2="8.41" y2="10.16" width="0" layer="19" extent="1-1"/>
+<wire x1="53.42" y1="10.16" x2="34.06" y2="14.3" width="0" layer="19" extent="16-16"/>
 </signal>
 <signal name="PDI-DATA">
@@
 <wire x1="56.74210625" y1="62.865" x2="56.13250625" y2="63.4746" width="0.4064" layer="16"/>
 </signal>
+<signal name="N$10">
+<contactref element="R1" pad="2"/>
+<contactref element="LED1" pad="A"/>
+<wire x1="49.85" y1="32" x2="49.75" y2="32" width="0.4064" layer="1"/>
+<wire x1="49.75" y1="32" x2="49.75" y2="29" width="0.4064" layer="1"/>
+</signal>
+<signal name="LED">
+<contactref element="R1" pad="1"/>
+<contactref element="IC1" pad="1"/>
+<wire x1="48.15" y1="32" x2="39" y2="32" width="0.4064" layer="1"/>
+<wire x1="39" y1="32" x2="31" y2="40" width="0.4064" layer="1"/>
+<via x="31" y="40" extent="1-16" drill="0.6"/>
+<wire x1="31" y1="40" x2="28.1" y2="40" width="0.4064" layer="16"/>
+<wire x1="28.1" y1="40" x2="25.59" y2="42.51" width="0.4064" layer="16"/>
+</signal>
 </signals>
