File: RemovingGround.sch (EAGLE design)
At the start: 34 parts, among them IC2 74AHC1G125DBV, IC3 74AHC1G125DBV, M1 HX1, X1 BU-SMA-V

Commit message: gf
Parts:
- added LED1: (no value), led:LEDCHIP-LED0603
- added R1: 220, resistor:R-US_R0603
Connections:
- new net LED: IC1.PA5/ADC5, R1.1
- new net N$10: LED1.A, R1.2
- net GND: now also LED1.C
Changed lines of the file:
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@@
 <?xml version="1.0" encoding="utf-8"?>
 <!DOCTYPE eagle SYSTEM "eagle.dtd">
-<eagle version="8.1.0">
+<eagle version="6.5.0">
 <drawing>
 <settings>
@@
 <part name="U$12" library="SHC" deviceset="CKN10160-ND" device=""/>
 <part name="GND13" library="SparkFun" deviceset="GND" device=""/>
+<part name="LED1" library="led" deviceset="LED" device="CHIP-LED0603"/>
+<part name="R1" library="resistor" deviceset="R-US_" device="R0603" value="220"/>
+<part name="GND16" library="SparkFun-Aesthetics" deviceset="GND" device=""/>
 </parts>
 <sheets>
@@
 <instance part="U$12" gate="G$1" x="-23.368" y="-30.48" rot="MR0"/>
 <instance part="GND13" gate="1" x="-7.62" y="180.34"/>
+<instance part="LED1" gate="G$1" x="119.38" y="137.16"/>
+<instance part="R1" gate="G$1" x="109.22" y="139.7"/>
+<instance part="GND16" gate="1" x="119.38" y="127"/>
 </instances>
 <busses>
@@
 <junction x="-7.62" y="190.5"/>
 <pinref part="GND13" gate="1" pin="GND"/>
+</segment>
+<segment>
+<pinref part="LED1" gate="G$1" pin="C"/>
+<wire x1="119.38" y1="132.08" x2="119.38" y2="129.54" width="0.1524" layer="91"/>
+<pinref part="GND16" gate="1" pin="GND"/>
 </segment>
 </net>
@@
 </segment>
 </net>
+<net name="N$10" class="0">
+<segment>
+<pinref part="R1" gate="G$1" pin="2"/>
+<pinref part="LED1" gate="G$1" pin="A"/>
+<wire x1="114.3" y1="139.7" x2="119.38" y2="139.7" width="0.1524" layer="91"/>
+</segment>
+</net>
+<net name="LED" class="0">
+<segment>
+<pinref part="R1" gate="G$1" pin="1"/>
+<wire x1="104.14" y1="139.7" x2="101.6" y2="139.7" width="0.1524" layer="91"/>
+<label x="101.6" y="139.7" size="1.778" layer="95"/>
+</segment>
+<segment>
+<pinref part="IC1" gate="G$1" pin="PA5/ADC5"/>
+<wire x1="48.26" y1="88.9" x2="35.56" y2="88.9" width="0.1524" layer="91"/>
+<label x="35.56" y="88.9" size="1.778" layer="95"/>
+</segment>
+</net>
